File: Hardware/PCB/Hardware.sch (KiCad schematic (older format))
At the start: 33 parts, among them J1 Conn_01x03_Male, M1 Motor_Servo, M2 Motor_Servo, M3 Motor_Servo, P1 Power, P2 Analog, P3 Digital, P4 Digital, P5 CONN_01X01, P6 CONN_01X01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

Commit message: Nouveau PCB simplifié
Parts:
- removed RV1: R_POT, Potentiometer_THT:Potentiometer_Alps_RK09L_Single_Vertical, symbol Device:R_POT
- removed SW1: SW_Push, Button_Switch_THT:SW_PUSH_6mm, symbol Switch:SW_Push
- added R11: R, Resistor_THT:R_Axial_DIN0204_L3.6mm_D1.6mm_P2.54mm_Vertical, symbol Device:R
- BZ1: footprint Buzzer_Beeper:MagneticBuzzer_Kingstate_KCG0601 -> Connector_PinHeader_2.54mm:PinHeader_1x02_P2.54mm_Horizontal
- R1: footprint Resistor_THT:R_Axial_DIN0204_L3.6mm_D1.6mm_P1.90mm_Vertical -> Resistor_THT:R_Axial_DIN0204_L3.6mm_D1.6mm_P2.54mm_Vertical
- R2, R4, R6, R8: footprint Connector_JST:JST_XH_B02B-XH-A_1x02_P2.50mm_Vertical -> Connector_PinHeader_2.54mm:PinHeader_1x02_P2.54mm_Vertical
Connections:
- wire segments 146 -> 148
Changed lines of the file:
@@
 	10200 2900 10550 2900
-Wire Wire Line
-	10200 2800 10550 2800
 Wire Wire Line
 	10200 2600 10550 2600
@@
 F 0 "R2" H 1820 5096 50  0000 L CNN
 F 1 "LDR03" H 1820 5005 50  0000 L CNN
-F 2 "Connector_JST:JST_XH_B02B-XH-A_1x02_P2.50mm_Vertical" V 1925 5050 50  0001 C CNN
+F 2 "Connector_PinHeader_2.54mm:PinHeader_1x02_P2.54mm_Vertical" V 1925 5050 50  0001 C CNN
 F 3 "http://www.elektronica-componenten.nl/WebRoot/StoreNL/Shops/61422969/54F1/BA0C/C664/31B9/2173/C0A8/2AB9/2AEF/LDR03IMP.pdf" H 1750 5000 50  0001 C CNN
 	1    1750 5050
@@
 F 0 "R4" H 2420 5096 50  0000 L CNN
 F 1 "LDR03" H 2420 5005 50  0000 L CNN
-F 2 "Connector_JST:JST_XH_B02B-XH-A_1x02_P2.50mm_Vertical" V 2525 5050 50  0001 C CNN
+F 2 "Connector_PinHeader_2.54mm:PinHeader_1x02_P2.54mm_Vertical" V 2525 5050 50  0001 C CNN
 F 3 "http://www.elektronica-componenten.nl/WebRoot/StoreNL/Shops/61422969/54F1/BA0C/C664/31B9/2173/C0A8/2AB9/2AEF/LDR03IMP.pdf" H 2350 5000 50  0001 C CNN
 	1    2350 5050
@@
 F 0 "R6" H 3070 5096 50  0000 L CNN
 F 1 "LDR03" H 3070 5005 50  0000 L CNN
-F 2 "Connector_JST:JST_XH_B02B-XH-A_1x02_P2.50mm_Vertical" V 3175 5050 50  0001 C CNN
+F 2 "Connector_PinHeader_2.54mm:PinHeader_1x02_P2.54mm_Vertical" V 3175 5050 50  0001 C CNN
 F 3 "http://www.elektronica-componenten.nl/WebRoot/StoreNL/Shops/61422969/54F1/BA0C/C664/31B9/2173/C0A8/2AB9/2AEF/LDR03IMP.pdf" H 3000 5000 50  0001 C CNN
 	1    3000 5050
@@
 F 0 "R8" H 3670 5096 50  0000 L CNN
 F 1 "LDR03" H 3670 5005 50  0000 L CNN
-F 2 "Connector_JST:JST_XH_B02B-XH-A_1x02_P2.50mm_Vertical" V 3775 5050 50  0001 C CNN
+F 2 "Connector_PinHeader_2.54mm:PinHeader_1x02_P2.54mm_Vertical" V 3775 5050 50  0001 C CNN
 F 3 "http://www.elektronica-componenten.nl/WebRoot/StoreNL/Shops/61422969/54F1/BA0C/C664/31B9/2173/C0A8/2AB9/2AEF/LDR03IMP.pdf" H 3600 5000 50  0001 C CNN
 	1    3600 5050
@@
 	5150 3000 5300 3000
 Wire Wire Line
-	5300 3000 5300 2450
+	5300 3000 5300 2900
 Connection ~ 5300 2450
 Wire Wire Line
@@
 	2650 6200 3000 6200
 Wire Wire Line
-	10200 1600 11200 1600
-Wire Wire Line
-	11200 1600 11200 4900
-Wire Wire Line
 	3600 4900 3000 4900
-Connection ~ 3600 4900
 Wire Wire Line
 	3000 4900 2350 4900
@@
 	1    0    0    -1
 $EndComp
-$Comp
-L Device:R R1
-U 1 1 5BE0B72B
-P 1650 1050
-F 0 "R1" V 1443 1050 50  0000 C CNN
-F 1 "R" V 1534 1050 50  0000 C CNN
-F 2 "Resistor_THT:R_Axial_DIN0204_L3.6mm_D1.6mm_P1.90mm_Vertical" V 1580 1050 50  0001 C CNN
-F 3 "~" H 1650 1050 50  0001 C CNN
-	1    1650 1050
-	0    1    1    0
-$EndComp
-Wire Wire Line
-	1200 1050 1500 1050
-$Comp
-L Switch:SW_Push SW1
-U 1 1 5BE11AD8
-P 2250 950
-F 0 "SW1" H 2250 1235 50  0000 C CNN
-F 1 "SW_Push" H 2250 1144 50  0000 C CNN
-F 2 "Button_Switch_THT:SW_PUSH_6mm" H 2250 1150 50  0001 C CNN
-F 3 "" H 2250 1150 50  0001 C CNN
-	1    2250 950
-	1    0    0    -1
-$EndComp
-Wire Wire Line
-	1200 950  2050 950
-Wire Wire Line
-	2450 950  9050 950
 Wire Wire Line
 	9050 950  9050 1350
@@
 Wire Wire Line
 	9050 1350 9050 2000
-Wire Wire Line
-	1800 1050 8700 1050
-Wire Wire Line
-	8700 1050 8700 2900
-Wire Wire Line
-	8700 2900 9400 2900
 Wire Wire Line
 	5300 2450 5300 1750
@@
 $EndComp
 Wire Wire Line
-	3600 4900 11200 4900
-Wire Wire Line
 	9350 4150 9800 4150
 Wire Wire Line
@@
 Wire Wire Line
 	9900 4100 9900 4250
-Wire Wire Line
-	9900 4100 9450 4100
 Wire Wire Line
 	9450 4100 9450 4250
@@
 F 0 "BZ1" V 8860 4452 50  0000 L CNN
 F 1 "Buzzer" V 8951 4452 50  0000 L CNN
-F 2 "Buzzer_Beeper:MagneticBuzzer_Kingstate_KCG0601" V 8875 4400 50  0001 C CNN
+F 2 "Connector_PinHeader_2.54mm:PinHeader_1x02_P2.54mm_Horizontal" V 8875 4400 50  0001 C CNN
 F 3 "~" V 8875 4400 50  0001 C CNN
 	1    8900 4300
@@
 Wire Wire Line
 	10200 2000 10950 2000
-$Comp
-L Device:R_POT RV1
-U 1 1 5BE52801
-P 9150 3900
-F 0 "RV1" H 9080 3946 50  0000 R CNN
-F 1 "R_POT" H 9080 3855 50  0000 R CNN
-F 2 "Potentiometer_THT:Potentiometer_Alps_RK09L_Single_Vertical" H 9150 3900 50  0001 C CNN
-F 3 "~" H 9150 3900 50  0001 C CNN
-	1    9150 3900
-	0    -1   -1   0
-$EndComp
-Wire Wire Line
-	9150 3750 9300 3750
-Wire Wire Line
-	9300 3750 9300 3900
-Wire Wire Line
-	9300 3900 10950 3900
 Wire Wire Line
 	10950 2000 10950 3900
-Connection ~ 9300 3900
-Wire Wire Line
-	9000 3850 8800 3850
-Wire Wire Line
-	9000 3850 9000 3900
 Wire Wire Line
 	11100 1800 11100 3500
@@
 Wire Wire Line
 	8800 4150 9050 4150
-Wire Wire Line
-	9000 4200 9000 4000
-Wire Wire Line
-	9000 4000 8800 4000
-Wire Wire Line
-	8800 4000 8800 3850
 $Comp
 L power:GND #PWR0102
@@
 $EndComp
 Wire Wire Line
-	7100 4200 7300 4200
-Wire Wire Line
-	7300 4200 7300 4300
-Wire Wire Line
-	7300 4200 7300 4050
-Connection ~ 7300 4200
-Wire Wire Line
 	7600 5950 11050 5950
 Wire Wire Line
@@
 	10900 4000 10900 2300
 Wire Wire Line
-	7600 4050 7600 4300
-Wire Wire Line
 	10200 2300 10900 2300
-Connection ~ 7600 4300
 Wire Wire Line
 	7600 4300 7600 5950
@@
 	1    0    0    -1
 $EndComp
+Wire Wire Line
+	1200 950  7200 950
+Wire Wire Line
+	8700 2900 9400 2900
+$Comp
+L Device:R R1
+U 1 1 5C168D50
+P 9100 3900
+F 0 "R1" H 9170 3946 50  0000 L CNN
+F 1 "R" H 9170 3855 50  0000 L CNN
+F 2 "Resistor_THT:R_Axial_DIN0204_L3.6mm_D1.6mm_P2.54mm_Vertical" V 9030 3900 50  0001 C CNN
+F 3 "~" H 9100 3900 50  0001 C CNN
+	1    9100 3900
+	0    -1   -1   0
+$EndComp
+Wire Wire Line
+	9000 4200 9000 4000
+Wire Wire Line
+	9000 4000 8950 4000
+Wire Wire Line
+	8950 3800 8950 3900
+Connection ~ 8950 3900
+Wire Wire Line
+	8950 3900 8950 4000
+Wire Wire Line
+	9250 3900 10950 3900
+Wire Wire Line
+	3600 4900 3600 2900
+Wire Wire Line
+	3600 2900 5300 2900
+Connection ~ 3600 4900
+Connection ~ 5300 2900
+Wire Wire Line
+	5300 2900 5300 2450
+$Comp
+L Device:R R11
+U 1 1 5C1A7B03
+P 6800 4350
+F 0 "R11" H 6870 4396 50  0000 L CNN
+F 1 "R" H 6870 4305 50  0000 L CNN
+F 2 "Resistor_THT:R_Axial_DIN0204_L3.6mm_D1.6mm_P2.54mm_Vertical" V 6730 4350 50  0001 C CNN
+F 3 "~" H 6800 4350 50  0001 C CNN
+	1    6800 4350
+	1    0    0    -1
+$EndComp
+$Comp
+L power:GND #PWR0103
+U 1 1 5C1A7B0A
+P 6800 4500
+F 0 "#PWR0103" H 6800 4250 50  0001 C CNN
+F 1 "GND" H 6805 4327 50  0000 C CNN
+F 2 "" H 6800 4500 50  0001 C CNN
+F 3 "" H 6800 4500 50  0001 C CNN
+	1    6800 4500
+	1    0    0    -1
+$EndComp
+Wire Wire Line
+	6800 4200 6800 4050
+Wire Wire Line
+	6800 4050 7300 4050
+Wire Wire Line
+	7100 4200 7300 4200
+Wire Wire Line
+	7300 4200 7300 4300
+Wire Wire Line
+	10600 2800 10600 3700
+Wire Wire Line
+	10600 3700 8450 3700
+Wire Wire Line
+	8450 3700 8450 4050
+Wire Wire Line
+	8450 4050 7600 4050
+Wire Wire Line
+	10200 2800 10600 2800
+Wire Wire Line
+	7200 6200 9700 6200
+Wire Wire Line
+	9700 6200 9700 4100
+Wire Wire Line
+	9450 4100 9700 4100
+Wire Wire Line
+	7200 950  7200 6200
+Connection ~ 7200 950
+Wire Wire Line
+	7200 950  9050 950
+Connection ~ 9700 4100
+Wire Wire Line
+	9700 4100 9900 4100
 $EndSCHEMATC

Commit message: PCB corrigé et verifié. Typon prêt
Parts:
- added R12, R13, R14: R, Resistor_THT:R_Axial_DIN0204_L3.6mm_D1.6mm_P5.08mm_Horizontal, symbol Device:R
- D1, D3: footprint Diode_THT:D_DO-15_P5.08mm_Vertical_KathodeUp -> Diode_THT:D_T-1_P10.16mm_Horizontal
- D2: footprint Diode_THT:D_A-405_P5.08mm_Vertical_KathodeUp -> Diode_THT:D_T-1_P10.16mm_Horizontal
- J1: footprint Connector_PinHeader_1.27mm:PinHeader_1x03_P1.27mm_Horizontal -> Connector_PinHeader_2.54mm:PinHeader_1x03_P2.54mm_Horizontal
- R3, R7: footprint Resistor_THT:R_Axial_DIN0204_L3.6mm_D1.6mm_P1.90mm_Vertical -> Resistor_THT:R_Axial_DIN0204_L3.6mm_D1.6mm_P5.08mm_Horizontal
Connections:
- wire segments 148 -> 169
Changed lines of the file:
@@
 F 0 "R3" H 1820 6096 50  0000 L CNN
 F 1 "R" H 1820 6005 50  0000 L CNN
-F 2 "Resistor_THT:R_Axial_DIN0204_L3.6mm_D1.6mm_P1.90mm_Vertical" V 1680 6050 50  0001 C CNN
+F 2 "Resistor_THT:R_Axial_DIN0204_L3.6mm_D1.6mm_P5.08mm_Horizontal" V 1680 6050 50  0001 C CNN
 F 3 "~" H 1750 6050 50  0001 C CNN
 	1    1750 6050
@@
 F 0 "R7" H 3070 6096 50  0000 L CNN
 F 1 "R" H 3070 6005 50  0000 L CNN
-F 2 "Resistor_THT:R_Axial_DIN0204_L3.6mm_D1.6mm_P1.90mm_Vertical" V 2930 6050 50  0001 C CNN
+F 2 "Resistor_THT:R_Axial_DIN0204_L3.6mm_D1.6mm_P5.08mm_Horizontal" V 2930 6050 50  0001 C CNN
 F 3 "~" H 3000 6050 50  0001 C CNN
 	1    3000 6050
@@
 F 0 "J1" H 1106 1328 50  0000 C CNN
 F 1 "Conn_01x03_Male" H 1106 1237 50  0000 C CNN
-F 2 "Connector_PinHeader_1.27mm:PinHeader_1x03_P1.27mm_Horizontal" H 1000 1050 50  0001 C CNN
+F 2 "Connector_PinHeader_2.54mm:PinHeader_1x03_P2.54mm_Horizontal" H 1000 1050 50  0001 C CNN
 F 3 "~" H 1000 1050 50  0001 C CNN
 	1    1000 1050
@@
 F 0 "D3" H 6200 2835 50  0000 C CNN
 F 1 "DIODE" H 6200 2926 50  0000 C CNN
-F 2 "Diode_THT:D_DO-15_P5.08mm_Vertical_KathodeUp" H 6200 3100 50  0001 C CNN
+F 2 "Diode_THT:D_T-1_P10.16mm_Horizontal" H 6200 3100 50  0001 C CNN
 F 3 "" H 6200 3100 50  0001 C CNN
 	1    6200 3100
@@
 F 0 "D2" H 6200 2285 50  0000 C CNN
 F 1 "DIODE" H 6200 2376 50  0000 C CNN
-F 2 "Diode_THT:D_A-405_P5.08mm_Vertical_KathodeUp" H 6200 2550 50  0001 C CNN
+F 2 "Diode_THT:D_T-1_P10.16mm_Horizontal" H 6200 2550 50  0001 C CNN
 F 3 "" H 6200 2550 50  0001 C CNN
 	1    6200 2550
@@
 F 0 "D1" H 6200 1585 50  0000 C CNN
 F 1 "DIODE" H 6200 1676 50  0000 C CNN
-F 2 "Diode_THT:D_DO-15_P5.08mm_Vertical_KathodeUp" H 6200 1850 50  0001 C CNN
+F 2 "Diode_THT:D_T-1_P10.16mm_Horizontal" H 6200 1850 50  0001 C CNN
 F 3 "" H 6200 1850 50  0001 C CNN
 	1    6200 1850
@@
 Wire Wire Line
 	9700 4100 9900 4100
+$Comp
+L Device:R R12
+U 1 1 5C147C7E
+P 1600 2950
+F 0 "R12" H 1670 2996 50  0000 L CNN
+F 1 "R" H 1670 2905 50  0000 L CNN
+F 2 "Resistor_THT:R_Axial_DIN0204_L3.6mm_D1.6mm_P5.08mm_Horizontal" V 1530 2950 50  0001 C CNN
+F 3 "~" H 1600 2950 50  0001 C CNN
+	1    1600 2950
+	1    0    0    -1
+$EndComp
+Wire Wire Line
+	1600 2200 1600 2800
+$Comp
+L Device:R R13
+U 1 1 5C14DD6D
+P 2450 2200
+F 0 "R13" H 2520 2246 50  0000 L CNN
+F 1 "R" H 2520 2155 50  0000 L CNN
+F 2 "Resistor_THT:R_Axial_DIN0204_L3.6mm_D1.6mm_P5.08mm_Horizontal" V 2380 2200 50  0001 C CNN
+F 3 "~" H 2450 2200 50  0001 C CNN
+	1    2450 2200
+	1    0    0    -1
+$EndComp
+Wire Wire Line
+	2450 2350 2550 2350
+Wire Wire Line
+	2450 1450 2450 1550
+$Comp
+L Device:R R14
+U 1 1 5C1543E2
+P 950 3900
+F 0 "R14" H 1020 3946 50  0000 L CNN
+F 1 "R" H 1020 3855 50  0000 L CNN
+F 2 "Resistor_THT:R_Axial_DIN0204_L3.6mm_D1.6mm_P5.08mm_Horizontal" V 880 3900 50  0001 C CNN
+F 3 "~" H 950 3900 50  0001 C CNN
+	1    950  3900
+	1    0    0    -1
+$EndComp
+Wire Wire Line
+	950  4050 1300 4050
+$Comp
+L power:GND #PWR?
+U 1 1 5C15ACC3
+P 1550 4050
+F 0 "#PWR?" H 1550 3800 50  0001 C CNN
+F 1 "GND" H 1555 3877 50  0000 C CNN
+F 2 "" H 1550 4050 50  0001 C CNN
+F 3 "" H 1550 4050 50  0001 C CNN
+	1    1550 4050
+	1    0    0    -1
+$EndComp
+Wire Wire Line
+	2200 3150 2200 3100
+Wire Wire Line
+	2200 2200 1900 2200
+Wire Wire Line
+	950  2200 950  3750
+Connection ~ 2200 3100
+Wire Wire Line
+	2200 3100 2200 3050
+Connection ~ 1600 2200
+Wire Wire Line
+	1600 2200 950  2200
+Wire Wire Line
+	1300 4050 1300 3100
+Wire Wire Line
+	1300 3100 1600 3100
+Connection ~ 1300 4050
+Wire Wire Line
+	1300 4050 1550 4050
+Connection ~ 1600 3100
+Wire Wire Line
+	1600 3100 2200 3100
+Wire Wire Line
+	2200 3050 2550 3050
+Wire Wire Line
+	2550 3050 2550 2350
+Connection ~ 2200 3050
+Wire Wire Line
+	2200 3050 2200 2200
+Connection ~ 2550 2350
+Wire Wire Line
+	2550 2350 3050 2350
+Wire Wire Line
+	1900 2200 1900 1550
+Wire Wire Line
+	1900 1550 2450 1550
+Connection ~ 1900 2200
+Wire Wire Line
+	1900 2200 1600 2200
+Connection ~ 2450 1550
+Wire Wire Line
+	2450 1550 2450 2050
 $EndSCHEMATC

Commit message: Code testeur UltraSon+Diodes sur PCB Ajout pull down sur la ligne ECHO
Parts:
- added R15: R, Resistor_THT:R_Axial_DIN0204_L3.6mm_D1.6mm_P2.54mm_Vertical, symbol Device:R
Connections:
- wire segments 169 -> 171
Changed lines of the file:
@@
 	950  4050 1300 4050
 $Comp
-L power:GND #PWR?
+L power:GND #PWR0104
 U 1 1 5C15ACC3
 P 1550 4050
-F 0 "#PWR?" H 1550 3800 50  0001 C CNN
+F 0 "#PWR0104" H 1550 3800 50  0001 C CNN
 F 1 "GND" H 1555 3877 50  0000 C CNN
 F 2 "" H 1550 4050 50  0001 C CNN
@@
 Wire Wire Line
 	2450 1550 2450 2050
+$Comp
+L Device:R R15
+U 1 1 5C154DF3
+P 6600 3850
+F 0 "R15" H 6670 3896 50  0000 L CNN
+F 1 "R" H 6670 3805 50  0000 L CNN
+F 2 "Resistor_THT:R_Axial_DIN0204_L3.6mm_D1.6mm_P2.54mm_Vertical" V 6530 3850 50  0001 C CNN
+F 3 "~" H 6600 3850 50  0001 C CNN
+	1    6600 3850
+	0    -1   -1   0
+$EndComp
+Wire Wire Line
+	6400 3650 6400 3850
+Wire Wire Line
+	6400 3850 6450 3850
+Connection ~ 6400 3650
+$Comp
+L power:GND #PWR0105
+U 1 1 5C16564B
+P 6750 3850
+F 0 "#PWR0105" H 6750 3600 50  0001 C CNN
+F 1 "GND" H 6755 3677 50  0000 C CNN
+F 2 "" H 6750 3850 50  0001 C CNN
+F 3 "" H 6750 3850 50  0001 C CNN
+	1    6750 3850
+	1    0    0    -1
+$EndComp
 $EndSCHEMATC

Commit message: Texte sur le pcb pour eviter erreur de gravure
Connections:
- wire segments 171 -> 157
Changed lines of the file:
@@
 Wire Wire Line
 	5150 3000 5300 3000
-Wire Wire Line
-	5300 3000 5300 2900
 Connection ~ 5300 2450
 Wire Wire Line
@@
 	3600 4900 3000 4900
 Wire Wire Line
-	3000 4900 2350 4900
+	3000 4900 2600 4900
 Wire Wire Line
 	2350 4900 2350 4950
@@
 Wire Wire Line
 	9250 3900 10950 3900
-Wire Wire Line
-	3600 4900 3600 2900
-Wire Wire Line
-	3600 2900 5300 2900
-Connection ~ 3600 4900
-Connection ~ 5300 2900
-Wire Wire Line
-	5300 2900 5300 2450
 $Comp
 L Device:R R11
@@
 L Device:R R12
 U 1 1 5C147C7E
-P 1600 2950
-F 0 "R12" H 1670 2996 50  0000 L CNN
-F 1 "R" H 1670 2905 50  0000 L CNN
-F 2 "Resistor_THT:R_Axial_DIN0204_L3.6mm_D1.6mm_P5.08mm_Horizontal" V 1530 2950 50  0001 C CNN
-F 3 "~" H 1600 2950 50  0001 C CNN
-	1    1600 2950
-	1    0    0    -1
-$EndComp
-Wire Wire Line
-	1600 2200 1600 2800
+P 850 3900
+F 0 "R12" H 920 3946 50  0000 L CNN
+F 1 "R" H 920 3855 50  0000 L CNN
+F 2 "Resistor_THT:R_Axial_DIN0204_L3.6mm_D1.6mm_P5.08mm_Horizontal" V 780 3900 50  0001 C CNN
+F 3 "~" H 850 3900 50  0001 C CNN
+	1    850  3900
+	1    0    0    -1
+$EndComp
 $Comp
 L Device:R R13
 U 1 1 5C14DD6D
-P 2450 2200
-F 0 "R13" H 2520 2246 50  0000 L CNN
-F 1 "R" H 2520 2155 50  0000 L CNN
-F 2 "Resistor_THT:R_Axial_DIN0204_L3.6mm_D1.6mm_P5.08mm_Horizontal" V 2380 2200 50  0001 C CNN
-F 3 "~" H 2450 2200 50  0001 C CNN
-	1    2450 2200
-	1    0    0    -1
-$EndComp
-Wire Wire Line
-	2450 2350 2550 2350
-Wire Wire Line
-	2450 1450 2450 1550
+P 750 3900
+F 0 "R13" H 820 3946 50  0000 L CNN
+F 1 "R" H 820 3855 50  0000 L CNN
+F 2 "Resistor_THT:R_Axial_DIN0204_L3.6mm_D1.6mm_P5.08mm_Horizontal" V 680 3900 50  0001 C CNN
+F 3 "~" H 750 3900 50  0001 C CNN
+	1    750  3900
+	1    0    0    -1
+$EndComp
 $Comp
 L Device:R R14
@@
 	1    0    0    -1
 $EndComp
-Wire Wire Line
-	950  4050 1300 4050
 $Comp
 L power:GND #PWR0104
@@
 	1    0    0    -1
 $EndComp
-Wire Wire Line
-	2200 3150 2200 3100
-Wire Wire Line
-	2200 2200 1900 2200
-Wire Wire Line
-	950  2200 950  3750
-Connection ~ 2200 3100
-Wire Wire Line
-	2200 3100 2200 3050
-Connection ~ 1600 2200
-Wire Wire Line
-	1600 2200 950  2200
-Wire Wire Line
-	1300 4050 1300 3100
-Wire Wire Line
-	1300 3100 1600 3100
-Connection ~ 1300 4050
-Wire Wire Line
-	1300 4050 1550 4050
-Connection ~ 1600 3100
-Wire Wire Line
-	1600 3100 2200 3100
-Wire Wire Line
-	2200 3050 2550 3050
-Wire Wire Line
-	2550 3050 2550 2350
-Connection ~ 2200 3050
-Wire Wire Line
-	2200 3050 2200 2200
-Connection ~ 2550 2350
-Wire Wire Line
-	2550 2350 3050 2350
-Wire Wire Line
-	1900 2200 1900 1550
-Wire Wire Line
-	1900 1550 2450 1550
-Connection ~ 1900 2200
-Wire Wire Line
-	1900 2200 1600 2200
-Connection ~ 2450 1550
-Wire Wire Line
-	2450 1550 2450 2050
 $Comp
 L Device:R R15
@@
 	1    0    0    -1
 $EndComp
+Wire Wire Line
+	650  4050 650  3750
+Wire Wire Line
+	650  3750 750  3750
+Wire Wire Line
+	650  4050 750  4050
+Connection ~ 750  4050
+Wire Wire Line
+	750  4050 850  4050
+Connection ~ 850  4050
+Wire Wire Line
+	850  4050 950  4050
+Connection ~ 950  4050
+Wire Wire Line
+	950  4050 1550 4050
+Connection ~ 750  3750
+Wire Wire Line
+	750  3750 850  3750
+Connection ~ 850  3750
+Wire Wire Line
+	850  3750 950  3750
+$Comp
+L power:+5V #PWR?
+U 1 1 5C18F55F
+P 2600 4700
+F 0 "#PWR?" H 2600 4550 50  0001 C CNN
+F 1 "+5V" H 2615 4873 50  0000 C CNN
+F 2 "" H 2600 4700 50  0001 C CNN
+F 3 "" H 2600 4700 50  0001 C CNN
+	1    2600 4700
+	1    0    0    -1
+$EndComp
+Wire Wire Line
+	5300 2450 5300 3000
+Wire Wire Line
+	2600 4700 2600 4900
+Connection ~ 2600 4900
+Wire Wire Line
+	2600 4900 2350 4900
 $EndSCHEMATC
